File: Hardware/ADS4242 Breakout.sch (KiCad schematic (older format))
At the start: 27 parts, among them P1 CONN_02X20, P2 CONN_02X20, U1 FOX924B, U2 SI5351A3, U3 ADS4242, U4 TPS734xxDRV

Commit message: Layout fertig.
Parts:
- added C20, C21, C22, C23, C24, C25, C26, C27, C30, C31, C32, C33, C34, C35, C36, C37, C38, C39: 47n, Capacitors_SMD:C_1206, symbol C
- added C28, C29: 3,3p, Capacitors_SMD:C_0402, symbol C
- added C40: 100n, Capacitors_SMD:C_0402, symbol C
- added D1, D2, D3, D4, D5: LED, LEDs:LED-0603, symbol LED
- added P10, P7, P8, P9: CONN_01X01, Mounting_Holes:MountingHole_3-5mm, symbol CONN_01X01
- added P3, P4, P5: BNC, Sockets_BNC:BNC_Socket_TYCO-AMP_LargePads, symbol BNC
- added P6: CONN_01X03, Pin_Headers:Pin_Header_Straight_1x03, symbol CONN_01X03
- added R10, R7, R8, R9: 15, Resistors_SMD:R_0603, symbol R
- added R11, R12, R13, R14, R3, R4, R5, R6: 25, Resistors_SMD:R_0402, symbol R
- added R15, R16, R17, R18, R19: 1k, Resistors_SMD:R_0402, symbol R
- added T1, T2: T1-1T-X65, Sockets_DIP:DIP-6__300_ELL, symbol T1-1T-X65
- added U5, U6: PLP-21.4, PhilippsFootprints:A01-8, symbol PLP-21.4
- P1, P2: footprint (none) -> Socket_Strips:Socket_Strip_Straight_2x20
- R2: footprint (none) -> Resistors_SMD:R_0603
- U1: footprint (none) -> PhilippsFootprints:FOX924
- U2: footprint (none) -> Housings_SSOP:MSOP-10_3x3mm_Pitch0.5mm
- U3: footprint (none) -> Housings_DFN_QFN:QFN-64-1EP_9x9mm_Pitch0.5mm
- U4: footprint (none) -> Housings_SOT-23_SOT-143_TSOT-6:SOT-23-6
Connections:
- net CTL05: now also R15.1
- net CTL06: now also R16.1
- net CTL07: now also R17.1
- net CTL08: now also R18.1
- net CTL09: now also R19.1
- net GND: now also D1.1 (K), D2.1 (K), D3.1 (K), D4.1 (K), D5.1 (K)
- net GNDA: now also C34.2, C35.2, C36.2, C37.2, C40.2, P3.2 (Ext), P4.2 (Ext), P5.2 (Ext), T1.6 (AB), T2.6 (AB), U5.2 (GND), U5.3 (GND), U5.4 (GND), U5.5 (GND), U5.6 (GND), U5.7 (GND), U6.2 (GND), U6.3 (GND), U6.4 (GND), U6.5 (GND), U6.6 (GND), U6.7 (GND)
- net PMode_0: now also P6.3 (P3)
- net PMode_1: now also P6.2 (P2)
- net PMode_2: now also P6.1 (P1)
- net VDD: now also C40.1
- net at U3.19 (IN_2+): now also R13.1, R9.1
- net at U3.20 (IN_2-): now also R10.2, R14.2
- net VCM: now reaches C9.1, U3.23 (VCM), U3.26 (Clk_In-)
- net VCM: now also C34.1, C35.1, C36.1, C37.1, R3.2, R4.1, R5.2, R6.1
- net at U3.29 (IN_1+): now also R11.1, R7.1
- net at U3.30 (IN_1-): now also R12.2, R8.2
- net at U2.9 (Clk1): now also C38.1, C39.1
- net 1,2V: no longer names the net of P1.2 (P2)
- net 1,2V: no longer P2.2 (P2)
- new net: D1.2 (A), R15.2
- new net: C38.2, C39.2, P5.1 (In)
- new net: D2.2 (A), R16.2
- new net: D3.2 (A), R17.2
- new net: D4.2 (A), R18.2
- new net: D5.2 (A), R19.2
- new net: P3.1 (In), U5.1 (In)
- new net: P4.1 (In), U6.1 (In)
- new net: C20.1, C21.1, U5.8 (Out)
- new net: C20.2, C21.2, T1.4 (AA)
- new net: C24.2, C25.2, R3.1, R7.2
- new net: C26.2, C27.2, R4.2, R8.1
- new net: C28.1, R11.2
- new net: C28.2, R12.1
- new net: C30.2, C31.2, R5.1, R9.2
- new net: C32.2, C33.2, R10.1, R6.2
- new net: C29.1, R13.2
- new net: C29.2, R14.1
- new net: C26.1, C27.1, T1.1 (SA)
- new net: C24.1, C25.1, T1.3 (SB)
- new net: C32.1, C33.1, T2.1 (SA)
- new net: C30.1, C31.1, T2.3 (SB)
- new net: C22.2, C23.2, T2.4 (AA)
- new net: C22.1, C23.1, U6.8 (Out)
- no-connect marks 8 -> 26
Other:
- note added: "Aus ESR-Gründen werden immer zwei der NP0-Kondensatoren parallel geschaltet\nso verschiebt sich die erste Resonanzfrequenz nach oben."
- note added: "IN: I"
- note added: "IN: Q"
